File: hardware/sensor-hat/sensor-hat.kicad_sch (KiCad schematic)
At the start: 67 parts, among them J10 probe socket, J11 data socket, J12 probe socket, J13 data socket, J14 probe socket, J16 I2C, J17 external, J3 EZO pH probe, J4 EZO ORP probe, J5 EZO I2C probe, J6 1-Wire, J7 Contacts, J8 4-20 mA, J9 data socket, P1 J1 + J2, SW1 TS-1187A, SW2 TS-1187A, SW3 SK13D07VG5, U1 EZO pH, U2 EZO ORP, U3 EZO I2C

Commit message: Show Poolveras on the display while button A is held, and put orderable part numbers on the hat BOM.
Parts:
- C10, C11, C3, C4, C5, C6, C7, C8, C9: LCSC C28233 -> (none); MPN (none) -> CL21B104KCFSFNE; Manufacturer (none) -> Samsung Electro-Mechanics; Package (none) -> 0805
- D1, D2, D3, D4, D5, D6, D7, D8: LCSC C7420333 -> (none); MPN (none) -> BAT54SLT1G; Manufacturer (none) -> onsemi; Package (none) -> SOT-23
- F1: MPN (none) -> MF-MSMF020-2; Manufacturer (none) -> Bourns; Package (none) -> 1812
- J10, J11, J12, J13, J14, J9: MPN (none) -> PPPC031LFBN-RC; Manufacturer (none) -> Sullins Connector Solutions; Package (none) -> 2.54mm
- J16: MPN (none) -> PPPC041LFBN-RC; Manufacturer (none) -> Sullins Connector Solutions; Package (none) -> 2.54mm
- J17: MPN (none) -> 68001-404HLF; Manufacturer (none) -> Amphenol; Package (none) -> 2.54mm
- J3, J4, J5: MPN (none) -> 1715721; Manufacturer (none) -> Phoenix Contact; Package (none) -> 5.08mm
- J6: MPN (none) -> 1715734; Manufacturer (none) -> Phoenix Contact; Package (none) -> 5.08mm
- J7, J8: MPN (none) -> 1715750; Manufacturer (none) -> Phoenix Contact; Package (none) -> 5.08mm
- R1, R2, R3, R4: LCSC C17471 -> (none); MPN (none) -> RC0805FR-07150RL; Manufacturer (none) -> Yageo; Package (none) -> 0805
- R10, R11, R12, R26, R5, R6, R7, R8, R9: LCSC C17513 -> (none); MPN (none) -> RC0805FR-071KL; Manufacturer (none) -> Yageo; Package (none) -> 0805
- R13, R14, R15, R16, R29, R30: LCSC C17414 -> (none); MPN (none) -> RC0805FR-0710KL; Manufacturer (none) -> Yageo; Package (none) -> 0805
- R17, R18, R19, R20, R21: LCSC C17408 -> (none); MPN (none) -> RC0805FR-07100RL; Manufacturer (none) -> Yageo; Package (none) -> 0805
- R24, R27, R28: LCSC C17673 -> (none); MPN (none) -> RC0805FR-074K7L; Manufacturer (none) -> Yageo; Package (none) -> 0805
- R25: LCSC C17520 -> (none); MPN (none) -> RC0805FR-072K2L; Manufacturer (none) -> Yageo; Package (none) -> 0805
- SW1, SW2: LCSC (none) -> C318884; MPN (none) -> TS-1187A-B-A-B; Manufacturer (none) -> XKB Connection; Package (none) -> 5.1x5.1mm
- SW3: MPN (none) -> SK13D07VG5; Manufacturer (none) -> SHOU HAN; Package (none) -> SP3T
